Commit message: Pure Pursuit tractor for forward and trailer for backward works, added restricted map of the environment

File: src/ridgeback/ridgeback_description/urdf/cart.urdf.xacro (robot description, xacro)
@@ -165,5 +165,5 @@
         <parent link="cargo_cart_bed_link"/>
         <child link="${prefix}_${side}_wheel_holder_link" />
-        <origin xyz="${-(location+0.05)} ${s_location*0.28} -0.0125" rpy="0 0 0" />
+        <origin xyz="${-(location)} ${s_location*0.28} -0.0125" rpy="0 0 0" />
         <axis xyz="0 0 1" />
         <!-- <limit lower="-${PI}" upper="${PI}" velocity="0" effort="0"/> -->
